Commit message: feat(sim): run the Piper on Gazebo Harmonic with the shared stack
backend:=gazebo spawns the same description into an in-process gz server
and runs the same controllers, MoveIt config and piper_py tests as mock.

Simulator models come from the official description through two tested
transforms in piper_description:
- robot_description(<sim>) gives the massless virtual gripper_link a 10 g
  placeholder inertial; SDFormat otherwise drops the gripper joint.
- physics_model() removes URDF mimic constraints (gz_ros2_control drives the
  mimic fingers itself) and widens joint limits by 0.01 rad / 2 mm, because
  DART velocity control cannot drive a joint off a limit it rests on: a
  gripper closed to zero never reopened.

piper_py no longer reports a gripper stall as success unless the fingers
stalled while closing (GRASPED). The integration test is parametrized by
backend, asserts which backend it runs against, and closes the gripper
onto its limit before reopening it. Gazebo transport is partitioned per
ROS_DOMAIN_ID.

Co-Authored-By: Claude Opus 5.5 <noreply@anthropic.com>
Claude-Session: https://claude.ai/code/session_01XJo9zxt3KewgHf4vEmzXbH

File: src/piper_description/urdf/piper.ros2_control.xacro (robot description, xacro)
@@ -22,5 +22,5 @@
   <xacro:macro name="piper_ros2_control" params="hardware gripper initial_positions_file controllers_file mujoco_model">
     <xacro:property name="init" value="${xacro.load_yaml(initial_positions_file)['initial_positions']}" />
-    <xacro:property name="known" value="${['mock', 'real']}" />
+    <xacro:property name="known" value="${['mock', 'real', 'gazebo']}" />
     <xacro:if value="${hardware not in known}">
       ${xacro.fatal('hardware:=' + hardware + ' is not implemented yet; supported: ' + ', '.join(known))}
@@ -40,4 +40,7 @@
           <param name="trigger_joint_command_threshold">-1</param>
         </xacro:if>
+        <xacro:if value="${hardware == 'gazebo'}">
+          <plugin>gz_ros2_control/GazeboSimSystem</plugin>
+        </xacro:if>
       </hardware>
       <xacro:piper_joint name="joint1" initial="${init['joint1']}" />
@@ -50,6 +53,25 @@
       <xacro:if value="${gripper}">
         <xacro:piper_joint name="gripper" initial="${init['gripper']}" />
+        <!-- Simulators must move the physical fingers. They follow `gripper` through the URDF mimic
+             relation (+/-0.5); ros2_control mimic joints carry state interfaces only. -->
+        <xacro:if value="${hardware == 'gazebo'}">
+          <joint name="gripper_joint1"><state_interface name="position" /><state_interface name="velocity" /></joint>
+          <joint name="gripper_joint2"><state_interface name="position" /><state_interface name="velocity" /></joint>
+        </xacro:if>
       </xacro:if>
     </ros2_control>
+    <xacro:if value="${hardware == 'gazebo'}">
+      <xacro:if value="${controllers_file == ''}">
+        ${xacro.fatal('hardware:=gazebo needs controllers_file:=/path/to/controllers.yaml')}
+      </xacro:if>
+      <!-- The controller manager runs inside Gazebo; the fingers follow `gripper` via URDF mimic. -->
+      <gazebo>
+        <plugin filename="gz_ros2_control-system" name="gz_ros2_control::GazeboSimROS2ControlPlugin">
+          <parameters>${controllers_file}</parameters>
+        </plugin>
+        <!-- Simulator ground truth for every joint, including the mimic fingers (gz topic .../joint_state). -->
+        <plugin filename="gz-sim-joint-state-publisher-system" name="gz::sim::systems::JointStatePublisher" />
+      </gazebo>
+    </xacro:if>
   </xacro:macro>
 </robot>

File: src/piper_description/urdf/piper.urdf.xacro (robot description, xacro)
@@ -3,6 +3,7 @@
   Piper Studio robot description.
   Geometry, limits and inertials come unmodified from the official AgileX
-  agx_arm_urdf model (see docs/description/DECISIONS.md). This file only adds
-  workspace frames (tcp_link, optional world anchor) and the ros2_control block
+  agx_arm_urdf model (see docs/description/DECISIONS.md). The official model is rooted at a
+  fixed `world` link (world -> base_link). This file only adds
+  workspace frames (tcp_link) and the ros2_control block
   that selects the hardware backend.
 -->
@@ -16,6 +17,4 @@
   <xacro:arg name="tcp_xyz" default="0 0 0.138" />
   <xacro:arg name="tcp_rpy" default="0 0 0" />
-  <!-- When set, add this link and fix base_link to it (simulators need a world anchor). -->
-  <xacro:arg name="world_link" default="" />
   <!-- Backend-specific inputs. -->
   <xacro:arg name="controllers_file" default="" />
@@ -41,12 +40,4 @@
     <origin xyz="$(arg tcp_xyz)" rpy="$(arg tcp_rpy)" />
   </joint>
-  <xacro:if value="${'$(arg world_link)' != ''}">
-    <link name="$(arg world_link)" />
-    <joint name="$(arg world_link)_to_base_joint" type="fixed">
-      <parent link="$(arg world_link)" />
-      <child link="base_link" />
-      <origin xyz="0 0 0" rpy="0 0 0" />
-    </joint>
-  </xacro:if>
   <xacro:include filename="$(find piper_description)/urdf/piper.ros2_control.xacro" />
   <xacro:piper_ros2_control

Commit message: feat(sim): add the MuJoCo backend generated from the official description
backend:=mujoco converts the simulator description to MJCF at launch
with mujoco_ros2_control's converter (run in the workspace venv, cached
by content hash) and drives it through mujoco_ros2_control with the same
controllers, MoveIt config and piper_py tests as mock and Gazebo.

piper_bringup/config/mujoco/inputs.xml adds what URDF cannot express:
position actuators named like the ros2_control joints, equality
constraints for the mimic fingers, gravity compensation, and contact
exclusions for world-link1 and finger-finger. The actuator model is
provisional. test_mujoco_model checks FK against the official URDF to
1e-6 m and the finger coupling.

piper_py now subscribes to joint states with latest-sample QoS in a
separate callback group: the reliable depth-10 queue in the shared group
could return states several hundred milliseconds old after an action.

Co-Authored-By: Claude Opus 5.5 <noreply@anthropic.com>
Claude-Session: https://claude.ai/code/session_01XJo9zxt3KewgHf4vEmzXbH

File: src/piper_description/urdf/piper.ros2_control.xacro (robot description, xacro)
@@ -20,7 +20,7 @@
     </joint>
   </xacro:macro>
-  <xacro:macro name="piper_ros2_control" params="hardware gripper initial_positions_file controllers_file mujoco_model">
+  <xacro:macro name="piper_ros2_control" params="hardware gripper initial_positions_file controllers_file mujoco_model mujoco_headless">
     <xacro:property name="init" value="${xacro.load_yaml(initial_positions_file)['initial_positions']}" />
-    <xacro:property name="known" value="${['mock', 'real', 'gazebo']}" />
+    <xacro:property name="known" value="${['mock', 'real', 'gazebo', 'mujoco']}" />
     <xacro:if value="${hardware not in known}">
       ${xacro.fatal('hardware:=' + hardware + ' is not implemented yet; supported: ' + ', '.join(known))}
@@ -42,4 +42,12 @@
         <xacro:if value="${hardware == 'gazebo'}">
           <plugin>gz_ros2_control/GazeboSimSystem</plugin>
+        </xacro:if>
+        <xacro:if value="${hardware == 'mujoco'}">
+          <!-- MJCF generated from this description by piper_description.mujoco_model();
+               the fingers follow `gripper` through MJCF equality constraints. -->
+          <plugin>mujoco_ros2_control/MujocoSystemInterface</plugin>
+          <param name="mujoco_model">${mujoco_model}</param>
+          <param name="headless">${mujoco_headless}</param>
+          <param name="sim_speed_factor">1.0</param>
         </xacro:if>
       </hardware>

File: src/piper_description/urdf/piper.urdf.xacro (robot description, xacro)
@@ -20,4 +20,5 @@
   <xacro:arg name="controllers_file" default="" />
   <xacro:arg name="mujoco_model" default="" />
+  <xacro:arg name="mujoco_headless" default="true" />
   <xacro:property name="use_gripper" value="$(arg gripper)" />
   <xacro:if value="${use_gripper}">
@@ -46,4 +47,5 @@
     initial_positions_file="$(arg initial_positions_file)"
     controllers_file="$(arg controllers_file)"
-    mujoco_model="$(arg mujoco_model)" />
+    mujoco_model="$(arg mujoco_model)"
+    mujoco_headless="$(arg mujoco_headless)" />
 </robot>

Commit message: feat(sim): add the Isaac Sim backend
backend:=isaac runs the shared controllers and MoveIt config; Isaac Sim 6.1
runs as its own headless process in its own environment (isaac/run_piper.py,
scripts/isaac.sh) and exchanges /isaac/joint_commands, /isaac/joint_states
and /clock with ros2_control's JointStateTopicSystem. The USD is generated
from the same description (export_urdf.py + Isaac's URDF importer).

Launch gates ros2_control on /clock (Isaac takes ~30 s to start). The runner
couples the fingers to the gripper width itself, paces to real time, and is
stopped through a PID file because gpu-run does not forward signals.
The Isaac integration test is opt-in so routine runs never use the GPU.

Co-Authored-By: Claude Sonnet 5.5 <noreply@anthropic.com>
Claude-Session: https://claude.ai/code/session_01XJo9zxt3KewgHf4vEmzXbH

File: src/piper_description/urdf/piper.ros2_control.xacro (robot description, xacro)
@@ -11,5 +11,5 @@
 -->
 <robot xmlns:xacro="http://www.ros.org/wiki/xacro">
-  <xacro:macro name="piper_joint" params="name initial">
+  <xacro:macro name="piper_joint" params="name initial effort:=false">
     <joint name="${name}">
       <command_interface name="position" />
@@ -18,9 +18,11 @@
       </state_interface>
       <state_interface name="velocity" />
+      <!-- Isaac's joint-state publisher always sends efforts; JointStateTopicSystem needs the interface. -->
+      <xacro:if value="${effort}"><state_interface name="effort" /></xacro:if>
     </joint>
   </xacro:macro>
   <xacro:macro name="piper_ros2_control" params="hardware gripper initial_positions_file controllers_file mujoco_model mujoco_headless">
     <xacro:property name="init" value="${xacro.load_yaml(initial_positions_file)['initial_positions']}" />
-    <xacro:property name="known" value="${['mock', 'real', 'gazebo', 'mujoco']}" />
+    <xacro:property name="known" value="${['mock', 'real', 'gazebo', 'mujoco', 'isaac']}" />
     <xacro:if value="${hardware not in known}">
       ${xacro.fatal('hardware:=' + hardware + ' is not implemented yet; supported: ' + ', '.join(known))}
@@ -43,4 +45,13 @@
           <plugin>gz_ros2_control/GazeboSimSystem</plugin>
         </xacro:if>
+        <xacro:if value="${hardware == 'isaac'}">
+          <!-- Isaac Sim runs as a separate process (isaac/run_piper.py) and exchanges joint states and
+               position targets over ROS topics, like the real driver. Its own ROS bridge publishes
+               /clock. The fingers are driven by the Isaac runner from `gripper`. -->
+          <plugin>joint_state_topic_hardware_interface/JointStateTopicSystem</plugin>
+          <param name="joint_commands_topic">isaac/joint_commands</param>
+          <param name="joint_states_topic">isaac/joint_states</param>
+          <param name="trigger_joint_command_threshold">-1</param>
+        </xacro:if>
         <xacro:if value="${hardware == 'mujoco'}">
           <!-- MJCF generated from this description by piper_description.mujoco_model();
@@ -52,18 +63,22 @@
         </xacro:if>
       </hardware>
-      <xacro:piper_joint name="joint1" initial="${init['joint1']}" />
-      <xacro:piper_joint name="joint2" initial="${init['joint2']}" />
-      <xacro:piper_joint name="joint3" initial="${init['joint3']}" />
-      <xacro:piper_joint name="joint4" initial="${init['joint4']}" />
-      <xacro:piper_joint name="joint5" initial="${init['joint5']}" />
-      <xacro:piper_joint name="joint6" initial="${init['joint6']}" />
+      <xacro:piper_joint name="joint1" initial="${init['joint1']}" effort="${hardware == 'isaac'}" />
+      <xacro:piper_joint name="joint2" initial="${init['joint2']}" effort="${hardware == 'isaac'}" />
+      <xacro:piper_joint name="joint3" initial="${init['joint3']}" effort="${hardware == 'isaac'}" />
+      <xacro:piper_joint name="joint4" initial="${init['joint4']}" effort="${hardware == 'isaac'}" />
+      <xacro:piper_joint name="joint5" initial="${init['joint5']}" effort="${hardware == 'isaac'}" />
+      <xacro:piper_joint name="joint6" initial="${init['joint6']}" effort="${hardware == 'isaac'}" />
       <!-- Gripper opening width in metres (official single-DOF model; fingers are URDF mimics). -->
       <xacro:if value="${gripper}">
-        <xacro:piper_joint name="gripper" initial="${init['gripper']}" />
-        <!-- Simulators must move the physical fingers. They follow `gripper` through the URDF mimic
-             relation (+/-0.5); ros2_control mimic joints carry state interfaces only. -->
+        <xacro:piper_joint name="gripper" initial="${init['gripper']}" effort="${hardware == 'isaac'}" />
+        <!-- Gazebo must be told about the mimic fingers (state interfaces only). Mock and Isaac leave
+             them out: the URDF mimic relation (+/-0.5) is enough for ros2_control, and Isaac's runner
+             couples the fingers to `gripper` in physics. -->
         <xacro:if value="${hardware == 'gazebo'}">
-          <joint name="gripper_joint1"><state_interface name="position" /><state_interface name="velocity" /></joint>
-          <joint name="gripper_joint2"><state_interface name="position" /><state_interface name="velocity" /></joint>
+          <xacro:property name="fe" value="${False}" />
+          <joint name="gripper_joint1"><state_interface name="position" /><state_interface name="velocity" />
+            <xacro:if value="${fe}"><state_interface name="effort" /></xacro:if></joint>
+          <joint name="gripper_joint2"><state_interface name="position" /><state_interface name="velocity" />
+            <xacro:if value="${fe}"><state_interface name="effort" /></xacro:if></joint>
         </xacro:if>
       </xacro:if>
