Commit message: feat: MoveIt Servo TCP control, simulated D435, step-response study
- Servo: config/servo.yaml, launch integration (servo:=true), piper_py servo_start,
  servo_twist, servo_to_pose (closed loop, reports Servo halts), tcp_pose; idempotent
  streaming/trajectory handover. test_8 checks a TCP move on every backend.
- Wrist camera: RealSense D435 at AgileX's mount pose (own placeholder bracket; their
  mesh has no license), simulated image/depth/camera_info on MuJoCo with the realsense
  driver's topics and optical frame; Gazebo sensor defined; piper_py.image/camera_info.
  The D435 xacro's 70x oversized inertia is corrected for simulators.
- Step-response study (piper stepresp, tools/step_analysis.py) and shared MuJoCo/Isaac
  servo gains with a consistency test; joint4 damping retuned (overshoot 31% -> 2%).
- Isaac model check (scripts/isaac.sh check): fingertip pose and mass vs the URDF.
- Demo: settle dwell between steps so end states compare settled poses.

Co-Authored-By: Claude Sonnet 5.5 <noreply@anthropic.com>
Claude-Session: https://claude.ai/code/session_01XJo9zxt3KewgHf4vEmzXbH

File: src/piper_bringup/config/moveit/piper.srdf.xacro (robot description, xacro)
@@ -5,5 +5,15 @@
   <xacro:arg name="effector_type" default="agx_gripper" />
   <xacro:arg name="revo2_type" default="left" />
+  <xacro:arg name="camera" default="none" />
   <xacro:include filename="$(find agx_arm_moveit)/config/agx_arm.srdf.xacro" />
+  <xacro:if value="${'$(arg camera)' != 'none'}">
+    <!-- wrist camera and its bracket are rigidly mounted on link6 -->
+    <xacro:macro name="never" params="a b"><disable_collisions link1="${a}" link2="${b}" reason="Adjacent" /></xacro:macro>
+    <xacro:never a="camera_link" b="link6" /> <xacro:never a="camera_link" b="link5" />
+    <xacro:never a="camera_link" b="flange_link" /> <xacro:never a="camera_link" b="gripper_base" />
+    <xacro:never a="camera_link" b="camera_bracket_link" />
+    <xacro:never a="camera_bracket_link" b="link6" /> <xacro:never a="camera_bracket_link" b="link5" />
+    <xacro:never a="camera_bracket_link" b="flange_link" /> <xacro:never a="camera_bracket_link" b="gripper_base" />
+  </xacro:if>
   <!-- joint2/joint3 sit 0.01 rad inside their hard stops, matching config/initial_positions.yaml. -->
   <group_state name="rest" group="arm">

File: src/piper_description/urdf/piper.ros2_control.xacro (robot description, xacro)
@@ -22,5 +22,5 @@
     </joint>
   </xacro:macro>
-  <xacro:macro name="piper_ros2_control" params="hardware gripper initial_positions_file controllers_file mujoco_model mujoco_headless">
+  <xacro:macro name="piper_ros2_control" params="hardware gripper initial_positions_file controllers_file mujoco_model mujoco_headless camera:=none">
     <xacro:property name="init" value="${xacro.load_yaml(initial_positions_file)['initial_positions']}" />
     <xacro:property name="known" value="${['mock', 'real', 'gazebo', 'mujoco', 'isaac']}" />
@@ -69,4 +69,13 @@
       <xacro:piper_joint name="joint5" initial="${init['joint5']}" effort="${hardware == 'isaac'}" />
       <xacro:piper_joint name="joint6" initial="${init['joint6']}" effort="${hardware == 'isaac'}" />
+      <!-- MuJoCo renders the MJCF camera named "camera" and publishes it through this sensor (topics as the RealSense driver). -->
+      <xacro:if value="${hardware == 'mujoco' and camera != 'none'}">
+        <sensor name="camera">
+          <param name="frame_name">camera_color_optical_frame</param>
+          <param name="info_topic">/camera/color/camera_info</param>
+          <param name="image_topic">/camera/color/image_raw</param>
+          <param name="depth_topic">/camera/aligned_depth_to_color/image_raw</param>
+        </sensor>
+      </xacro:if>
       <!-- Gripper opening width in metres (official single-DOF model; fingers are URDF mimics). -->
       <xacro:if value="${gripper}">

File: src/piper_description/urdf/piper.urdf.xacro (robot description, xacro)
@@ -17,4 +17,12 @@
   <xacro:arg name="tcp_xyz" default="0 0 0.138" />
   <xacro:arg name="tcp_rpy" default="0 0 0" />
+  <!-- Wrist camera: none | d435 (RealSense D435 at AgileX's mount pose; see piper.camera.xacro). Simulated size/FOV
+       follow the D435 colour stream at 640x480 (69.4 deg horizontal). -->
+  <xacro:arg name="camera" default="none" />
+  <xacro:arg name="camera_bracket_mesh" default="" />
+  <xacro:arg name="camera_width" default="640" />
+  <xacro:arg name="camera_height" default="480" />
+  <xacro:arg name="camera_hfov_deg" default="69.4" />
+  <xacro:arg name="camera_rate" default="30" />
   <!-- Backend-specific inputs. -->
   <xacro:arg name="controllers_file" default="" />
@@ -41,4 +49,10 @@
     <origin xyz="$(arg tcp_xyz)" rpy="$(arg tcp_rpy)" />
   </joint>
+  <xacro:if value="${'$(arg camera)' == 'd435'}">
+    <xacro:include filename="$(find piper_description)/urdf/piper.camera.xacro" />
+    <xacro:piper_camera parent="link6" hardware="$(arg hardware)" bracket_mesh="$(arg camera_bracket_mesh)"
+                        width="$(arg camera_width)" height="$(arg camera_height)"
+                        hfov_deg="$(arg camera_hfov_deg)" update_rate="$(arg camera_rate)" />
+  </xacro:if>
   <xacro:include filename="$(find piper_description)/urdf/piper.ros2_control.xacro" />
   <xacro:piper_ros2_control
@@ -48,4 +62,5 @@
     controllers_file="$(arg controllers_file)"
     mujoco_model="$(arg mujoco_model)"
-    mujoco_headless="$(arg mujoco_headless)" />
+    mujoco_headless="$(arg mujoco_headless)"
+    camera="$(arg camera)" />
 </robot>

Commit message: ROS side for the real arm: zero/rest poses, guard limit clamp, canbus/speed_percent launch args, piper enable/disable/zero/rest, tests; arm_zero --rest; docs
Co-Authored-By: Claude Sonnet 5.5 <noreply@anthropic.com>
Claude-Session: https://claude.ai/code/session_01XJo9zxt3KewgHf4vEmzXbH

File: src/piper_bringup/config/moveit/piper.srdf.xacro (robot description, xacro)
@@ -16,5 +16,15 @@
     <xacro:never a="camera_bracket_link" b="flange_link" /> <xacro:never a="camera_bracket_link" b="gripper_base" />
   </xacro:if>
-  <!-- joint2/joint3 sit 0.01 rad inside their hard stops, matching config/initial_positions.yaml. -->
+  <!-- zero: all joints 0, with joint2/joint3 0.01 rad inside their hard stops (matches config/initial_positions.yaml). Start and end pose of every simulation. -->
+  <group_state name="zero" group="arm">
+    <joint name="joint1" value="0" />
+    <joint name="joint2" value="0.01" />
+    <joint name="joint3" value="-0.01" />
+    <joint name="joint4" value="0" />
+    <joint name="joint5" value="0" />
+    <joint name="joint6" value="0" />
+  </group_state>
+  <!-- rest: zero with joint5 lowered 16.82 deg (recorded on the real arm 2026-10-14): the wrist hangs just above the support brackets, so
+       disabling the motors there drops the arm only a few millimetres. Reach it from zero (piper rest does). -->
   <group_state name="rest" group="arm">
     <joint name="joint1" value="0" />
@@ -22,5 +32,5 @@
     <joint name="joint3" value="-0.01" />
     <joint name="joint4" value="0" />
-    <joint name="joint5" value="0" />
+    <joint name="joint5" value="0.2936" />
     <joint name="joint6" value="0" />
   </group_state>
